File: Coin Cell Solid PCB/Coin Cell Solid PCB.kicad_sch (KiCad schematic)
At the start: 51 parts, among them J1 0473461001, J4 UJ2-MIBV-4-SMT-TR-67, Q2 Q_PMOS_GSD, SW1 5136TR, U1 BQ21040DBVR, U2 TLV74010PDBVR, U3 LTC6992CS6-3#TRMPBF, U4 AP2502KTR-G1, U5 AP2502KTR-G1, U6 LTC2954CTS8-1#TRMPBF

Commit message: Added Coin cell holder
Parts:
- BT1: footprint (none) -> Dylan Library:Keystone_3047
Changed lines of the file:
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@@
 			)
 		)
-		(property "Footprint" ""
+		(property "Footprint" "Dylan Library:Keystone_3047"
 			(at 135.89 64.516 90)
 			(hide yes)

Commit message: initial layout of solid PCB done
Parts:
- D10, D3, D4, D5, D6, D7, D8, D9: footprint _Dylan_IC:BroadCom_ASMD-CWG7-NX7J2 -> Dylan Library:BroadCom_ASMD-CWG7-NX7J2
- J1: footprint _Dylan_IC:Molex_0473461001 -> Dylan Library:Molex_0473461001
- J4: footprint _Dylan_IC:SameSky_UJ2-MIBV-4-SMT-TR-67 -> Dylan Library:SameSky_UJ2-MIBV-4-SMT-TR-67
- RV1: footprint _Dylan_IC:Bourns_TC33X-2-104E -> Dylan Library:Bourns_TC33X-2-104E
- SW1: footprint _Dylan_IC:Keystone_5136TR -> Dylan Library:Keystone_5136TR
Changed lines of the file:
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@@
 			)
 		)
-		(property "Footprint" "_Dylan_IC:BroadCom_ASMD-CWG7-NX7J2"
+		(property "Footprint" "Dylan Library:BroadCom_ASMD-CWG7-NX7J2"
 			(at 267.97 121.92 0)
 			(hide yes)
@@
 			)
 		)
-		(property "Footprint" "_Dylan_IC:Molex_0473461001"
+		(property "Footprint" "Dylan Library:Molex_0473461001"
 			(at 21.59 55.88 0)
 			(hide yes)
@@
 			)
 		)
-		(property "Footprint" "_Dylan_IC:BroadCom_ASMD-CWG7-NX7J2"
+		(property "Footprint" "Dylan Library:BroadCom_ASMD-CWG7-NX7J2"
 			(at 204.47 123.19 0)
 			(hide yes)
@@
 			)
 		)
-		(property "Footprint" "_Dylan_IC:Keystone_5136TR"
+		(property "Footprint" "Dylan Library:Keystone_5136TR"
 			(at 167.64 78.74 0)
 			(hide yes)
@@
 			)
 		)
-		(property "Footprint" "_Dylan_IC:BroadCom_ASMD-CWG7-NX7J2"
+		(property "Footprint" "Dylan Library:BroadCom_ASMD-CWG7-NX7J2"
 			(at 198.12 123.19 0)
 			(hide yes)
@@
 			)
 		)
-		(property "Footprint" "_Dylan_IC:BroadCom_ASMD-CWG7-NX7J2"
+		(property "Footprint" "Dylan Library:BroadCom_ASMD-CWG7-NX7J2"
 			(at 260.35 121.92 0)
 			(hide yes)
@@
 			)
 		)
-		(property "Footprint" "_Dylan_IC:BroadCom_ASMD-CWG7-NX7J2"
+		(property "Footprint" "Dylan Library:BroadCom_ASMD-CWG7-NX7J2"
 			(at 182.88 123.19 0)
 			(hide yes)
@@
 			)
 		)
-		(property "Footprint" "_Dylan_IC:BroadCom_ASMD-CWG7-NX7J2"
+		(property "Footprint" "Dylan Library:BroadCom_ASMD-CWG7-NX7J2"
 			(at 252.73 121.92 0)
 			(hide yes)
@@
 			)
 		)
-		(property "Footprint" "_Dylan_IC:BroadCom_ASMD-CWG7-NX7J2"
+		(property "Footprint" "Dylan Library:BroadCom_ASMD-CWG7-NX7J2"
 			(at 274.32 121.92 0)
 			(hide yes)
@@
 			)
 		)
-		(property "Footprint" "_Dylan_IC:BroadCom_ASMD-CWG7-NX7J2"
+		(property "Footprint" "Dylan Library:BroadCom_ASMD-CWG7-NX7J2"
 			(at 190.5 123.19 0)
 			(hide yes)
@@
 			)
 		)
-		(property "Footprint" "_Dylan_IC:SameSky_UJ2-MIBV-4-SMT-TR-67"
+		(property "Footprint" "Dylan Library:SameSky_UJ2-MIBV-4-SMT-TR-67"
 			(at 21.59 26.67 0)
 			(hide yes)
@@
 			)
 		)
-		(property "Footprint" "_Dylan_IC:Bourns_TC33X-2-104E"
+		(property "Footprint" "Dylan Library:Bourns_TC33X-2-104E"
 			(at 68.58 127 0)
 			(hide yes)
