File: Coin Cell Solid PCB/Coin Cell Solid PCB.kicad_sch (KiCad schematic)
At the start: 51 parts, among them J1 0473461001, J4 UJ2-MIBV-4-SMT-TR-67, Q2 Q_PMOS_GSD, SW1 5136TR, U1 BQ21040DBVR, U2 TLV74010PDBVR, U3 LTC6992CS6-3#TRMPBF, U4 AP2502KTR-G1, U5 AP2502KTR-G1, U6 LTC2954CTS8-1#TRMPBF

Commit message: Added silk screen final touches, all PCBs 0.8mm, updated Fmod,
Parts:
- R4: value 10kΩ -> 500kΩ
Changed lines of the file:
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@@
 			)
 		)
-		(property "Value" "10kΩ"
+		(property "Value" "500kΩ"
 			(at 81.28 139.6999 0)
 			(show_name no)
