File: Coin Cell Solid PCB/_restore_backup_2026-09-28T21-58-23-549/Coin Cell Solid PCB.kicad_sch (KiCad schematic)
At the start: 51 parts, among them J1 0473461001, J4 UJ2-MIBV-4-SMT-TR-67, Q2 Q_PMOS_GSD, SW1 5136TR, U1 BQ21040DBVR, U2 TLV74010PDBVR, U3 LTC6992CS6-3#TRMPBF, U4 AP2502KTR-G1, U5 AP2502KTR-G1, U6 LTC2954CTS8-1#TRMPBF

Commit message: 0 DRC on Solid PCB
Parts:
- TP7: footprint Dylan Library:Harwin_S2761-46R -> TestPoint:TestPoint_Pad_D1.0mm
Changed lines of the file:
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@@
 			)
 		)
-		(property "Footprint" "Dylan Library:Harwin_S2761-46R"
+		(property "Footprint" "TestPoint:TestPoint_Pad_D1.0mm"
 			(at 77.47 27.94 0)
 			(hide yes)
