File: Coin Cell Battery Charger/Coin Cell Battery Charger.kicad_pcb (KiCad board)
At the start: 4 copper layers, 60 x 60 mm, 52 parts, among them J1 0473461001, J4 UJ2-MIBV-4-SMT-TR-67, Q2 Q_PMOS_GSD, SW1 5136TR, U1 BQ21040DBVR, U2 TLV74010PDBVR, U3 LTC6992CS6-3#TRMPBF, U4 AP2502KTR-G1, U5 AP2502KTR-G1, U6 LTC2954CTS8-1#TRMPBF

Commit message: Added silk screen final touches, all PCBs 0.8mm, updated Fmod,
Other:
- board text added: "Rev: SN:"
Changed lines of the file:
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@@
 	(generator_version "10.0")
 	(general
-		(thickness 1.6062)
+		(thickness 0.7912)
 		(legacy_teardrops no)
 	)
@@
 			(layer "dielectric 2"
 				(type "core")
-				(thickness 1.065)
+				(thickness 0.25)
 				(material "FR4")
 				(epsilon_r 4.5)
@@
 		(capping no)
 		(filling no)
+		(zone_defaults)
 		(grid_origin 150 100)
 		(pcbplotparams
@@
 		)
 	)
+	(gr_poly
+		(pts
+			(xy 125.5906 84.7092) (xy 134.881405 75.418395) (xy 139.825416 80.33953) (xy 130.507372 89.625972)
+		)
+		(stroke
+			(width 0.1)
+			(type solid)
+		)
+		(fill yes)
+		(layer "F.SilkS")
+	)
 	(gr_arc
 		(start 146 121.5)
@@
 		(layer "Edge.Cuts")
 	)
+	(gr_text "Rev:\nSN:"
+		(at 126.0732 92.0752 45)
+		(layer "F.SilkS")
+		(effects
+			(font
+				(face "Arial")
+				(size 1.5 1.5)
+				(thickness 0.2)
+			)
+			(justify left bottom)
+		)
+		(render_cache "Rev:\nSN:" 45
+			(polygon
+				(pts
+					(xy 124.096471 88.255269) (xy 124.170616 88.280358) (xy 124.238129 88.318443) (xy 124.300026 88.370355)
+					(xy 124.350333 88.430174) (xy 124.385819 88.493268) (xy 124.407777 88.560531) (xy 124.416538 88.633235)
+					(xy 124.410966 88.704761) (xy 124.389566 88.781507) (xy 124.349919 88.865156) (xy 124.288563 88.957317)
+					(xy 124.368741 88.934275) (xy 124.426771 88.926101) (xy 124.547853 88.93015) (xy 124.686477 88.952395)
+					(xy 125.163728 89.060229) (xy 124.986985 89.236971) (xy 124.622554 89.153749) (xy 124.372951 89.106989)
+					(xy 124.286363 89.101055) (xy 124.229627 89.106406) (xy 124.179754 89.121034) (xy 124.136884 89.141897)
+					(xy 124.053532 89.215016) (xy 123.890519 89.378029) (xy 124.368223 89.855733) (xy 124.227619 89.996337)
+					(xy 123.16237 88.931088) (xy 123.183807 88.909651) (xy 123.422141 88.909651) (xy 123.771352 89.258862)
+					(xy 124.073479 88.956735) (xy 124.158768 88.860186) (xy 124.204434 88.786274) (xy 124.222165 88.736023)
+					(xy 124.228307 88.687747) (xy 124.223604 88.640294) (xy 124.19925 88.573528) (xy 124.157155 88.517371)
+					(xy 124.103488 88.47614) (xy 124.044981 88.453732) (xy 123.979312 88.44898) (xy 123.914797 88.463402)
+					(xy 123.842186 88.502363) (xy 123.758335 88.573457) (xy 123.422141 88.909651) (xy 123.183807 88.909651)
+					(xy 123.633339 88.460119) (xy 123.732527 88.368653) (xy 123.812881 88.308547) (xy 123.877761 88.27269)
+					(xy 123.947062 88.250677) (xy 124.01936 88.244736)
+				)
+			)
+			(polygon
+				(pts
+					(xy 125.261849 87.707) (xy 125.358259 87.742531) (xy 125.456854 87.802365) (xy 125.559051 87.890708)
+					(xy 125.593053 87.926264) (xy 125.019238 88.500079) (xy 125.090298 88.555244) (xy 125.157412 88.59224)
+					(xy 125.221602 88.613747) (xy 125.284061 88.621513) (xy 125.367799 88.612175) (xy 125.442876 88.581384)
+					(xy 125.511903 88.527604) (xy 125.554151 88.476634) (xy 125.582045 88.423693) (xy 125.597068 88.36783)
+					(xy 125.59897 88.30985) (xy 125.586953 88.244052) (xy 125.558339 88.168225) (xy 125.709759 88.050094)
+					(xy 125.756188 88.152832) (xy 125.777278 88.252544) (xy 125.775041 88.351638) (xy 125.758322 88.423729)
+					(xy 125.727902 88.494783) (xy 125.682471 88.565694) (xy 125.619995 88.637121) (xy 125.529714 88.713292)
+					(xy 125.4387 88.76421) (xy 125.345546 88.792971) (xy 125.24831 88.800911) (xy 125.152116 88.788042)
+					(xy 125.056126 88.75354) (xy 124.958507 88.694966) (xy 124.857844 88.608236) (xy 124.767786 88.50403)
+					(xy 124.706786 88.403435) (xy 124.670564 88.305008) (xy 124.656491 88.206889) (xy 124.659765 88.157927)
+					(xy 124.827081 88.157927) (xy 124.83584 88.234914) (xy 124.865186 88.309599) (xy 124.917687 88.384021)
+					(xy 125.347336 87.954372) (xy 125.274419 87.902187) (xy 125.210937 87.872368) (xy 125.154661 87.860269)
+					(xy 125.088259 87.861319) (xy 125.027823 87.876013) (xy 124.971737 87.904344) (xy 124.918853 87.947636)
+					(xy 124.868146 88.011898) (xy 124.838067 88.081285) (xy 124.827081 88.157927) (xy 124.659765 88.157927)
+					(xy 124.663184 88.106797) (xy 124.690076 88.013599) (xy 124.737776 87.925239) (xy 124.808623 87.840257)
+					(xy 124.890881 87.771787) (xy 124.976774 87.725628) (xy 125.067737 87.699592) (xy 125.1658 87.693176)
+				)
+			)
+			(polygon
+				(pts
+					(xy 126.31887 87.905086) (xy 125.255176 87.426864) (xy 125.392865 87.289174) (xy 126.019917 87.585926)
+					(xy 126.224638 87.692075) (xy 126.126519 87.49681) (xy 125.826853 86.855186) (xy 125.960916 86.721123)
+					(xy 126.440563 87.783393)
+				)
+			)
+			(polygon
+				(pts
+					(xy 126.261554 86.718921) (xy 126.112336 86.569703) (xy 126.260841 86.421198) (xy 126.410059 86.570416)
+				)
+			)
+			(polygon
+				(pts
+					(xy 126.883294 87.340662) (xy 126.734077 87.191444) (xy 126.882582 87.042939) (xy 127.0318 87.192157)
+				)
+			)
+			(polygon
+				(pts
+					(xy 125.614723 91.483437) (xy 125.735703 91.339142) (xy 125.798564 91.382768) (xy 125.857311 91.411941)
+					(xy 125.912835 91.428711) (xy 125.970223 91.434062) (xy 126.033376 91.42709) (xy 126.103955 91.406108)
+					(xy 126.170769 91.374401) (xy 126.235695 91.331135) (xy 126.299156 91.275154) (xy 126.370341 91.191383)
+					(xy 126.417157 91.109227) (xy 126.437394 91.051249) (xy 126.44551 90.999252) (xy 126.443063 90.951849)
+					(xy 126.421755 90.885209) (xy 126.381925 90.83048) (xy 126.327309 90.790583) (xy 126.265414 90.771998)
+					(xy 126.196861 90.775085) (xy 126.106934 90.804704) (xy 126.033401 90.842727) (xy 125.86588 90.941875)
+					(xy 125.693503 91.038961) (xy 125.594322 91.080407) (xy 125.516407 91.09846) (xy 125.446073 91.10274)
+					(xy 125.381765 91.094655) (xy 125.320296 91.07447) (xy 125.263955 91.042985) (xy 125.211887 90.999386)
+					(xy 125.164452 90.941877) (xy 125.129532 90.876862) (xy 125.106709 90.80302) (xy 125.098808 90.726306)
+					(xy 125.107355 90.646936) (xy 125.133586 90.563196) (xy 125.173167 90.48385) (xy 125.225638 90.406904)
+					(xy 125.292195 90.331922) (xy 125.374705 90.258439) (xy 125.456647 90.202336) (xy 125.53856 90.16172)
+					(xy 125.625103 90.135189) (xy 125.708092 90.126601) (xy 125.789199 90.134907) (xy 125.867483 90.158714)
+					(xy 125.940307 90.196738) (xy 126.008686 90.249994) (xy 125.884079 90.394938) (xy 125.8059 90.344475)
+					(xy 125.731376 90.319324) (xy 125.657986 90.31599) (xy 125.58618 90.333599) (xy 125.508145 90.375901)
+					(xy 125.421271 90.449469) (xy 125.343369 90.539933) (xy 125.299844 90.616303) (xy 125.282156 90.682104)
+					(xy 125.283374 90.749603) (xy 125.301624 90.805562) (xy 125.336624 90.853148) (xy 125.377653 90.884769)
+					(xy 125.422262 90.902098) (xy 125.472176 90.90606) (xy 125.52322 90.894897) (xy 125.61289 90.855375)
+					(xy 125.759861 90.769925) (xy 125.95735 90.652677) (xy 126.0627 90.602573) (xy 126.154127 90.576422)
+					(xy 126.235186 90.567665) (xy 126.308029 90.574077) (xy 126.377895 90.595179) (xy 126.442677 90.630408)
+					(xy 126.503424 90.681003) (xy 126.553254 90.741505) (xy 126.590253 90.810507) (xy 126.614754 90.889481)
+					(xy 126.623986 90.971492) (xy 126.616768 91.056332) (xy 126.592022 91.145625) (xy 126.552918 91.230271)
+					(xy 126.499048 91.312202) (xy 126.428944 91.39199) (xy 126.328147 91.482352) (xy 126.233897 91.547558)
+					(xy 126.145081 91.5914) (xy 126.050877 91.618945) (xy 125.958125 91.627319) (xy 125.865103 91.617112)
+					(xy 125.775459 91.589392) (xy 125.692398 91.54523)
+				)
+			)
+			(polygon
+				(pts
+					(xy 126.995506 90.792269) (xy 125.930256 89.72702) (xy 126.074487 89.582789) (xy 127.468741 89.861277)
+					(xy 126.63237 89.024906) (xy 126.767145 88.890131) (xy 127.832395 89.95538) (xy 127.688229 90.099546)
+					(xy 126.293198 89.82041) (xy 127.130281 90.657494)
+				)
+			)
+			(polygon
+				(pts
+					(xy 127.46628 89.078013) (xy 127.317062 88.928795) (xy 127.465568 88.78029) (xy 127.614785 88.929508)
+				)
+			)
+			(polygon
+				(pts
+					(xy 128.088021 89.699754) (xy 127.938803 89.550536) (xy 128.087308 89.402031) (xy 128.236526 89.551248)
+				)
+			)
+		)
+	)
 	(gr_text "The Future is LIT"
 		(at 150 78.8418 0)
@@
 	)
 	(zone
+		(net "VBUS")
+		(layer "F.Cu")
+		(hatch none 0.1)
+		(priority 30000)
+		(attr
+			(teardrop
+				(type padvia)
+			)
+		)
+		(connect_pads yes
+			(clearance 0)
+		)
+		(min_thickness 0.0254)
+		(fill yes
+			(island_removal_mode 1)
+		)
+		(polygon
+			(pts
+				(xy 134.655863 118.867114) (xy 134.476258 118.687509) (xy 134.237234 118.868434) (xy 133.930901 119.412471)
+				(xy 134.589398 119.072172)
+			)
+		)
+	)
+	(zone
 		(net "GND")
 		(layer "F.Cu")
@@
 			)
 		)
-	)
-	(zone
-		(net "VBUS")
-		(layer "F.Cu")
-		(hatch none 0.1)
-		(priority 30000)
-		(attr
-			(teardrop
-				(type padvia)
-			)
-		)
-		(connect_pads yes
-			(clearance 0)
-		)
-		(min_thickness 0.0254)
-		(fill yes
-			(island_removal_mode 1)
-		)
-		(polygon
-			(pts
-				(xy 134.655863 118.867114) (xy 134.476258 118.687509) (xy 134.237234 118.868434) (xy 133.930901 119.412471)
-				(xy 134.589398 119.072172)
-			)
-		)
